Commit message: [UPD] description

File: robots/hsrb4s.urdf (robot description, URDF)
Before this commit: robot hsrb, 45 links, 44 joints
Links:
- link torso_lift_link: geometry collision mesh filename=package://hsr_meshes/meshes/torso_v0/torso.stl; visual mesh filename=package://hsr_meshes/meshes/torso_v0/torso_light.dae
Joints:
- joint arm_lift_joint: origin xyz=0.0 0.0 0.340 rpy=0.0 0.0 0.0 -> (none)
- joint base_imu_frame_joint: origin xyz=0.0005 0.1296 0.181 rpy=3.14159265359 0.0 0.0 -> (none)
- joint base_l_drive_wheel_joint: origin xyz=-0.11 0.133 0.04 rpy=0.0 0.0 0.0 -> (none)
- joint base_l_passive_wheel_x_frame_joint: origin xyz=0.1495                 0.055                 0.03 rpy=0.0 0.0 0.0 -> (none)
- joint base_r_drive_wheel_joint: origin xyz=-0.11 -0.133 0.04 rpy=0.0 0.0 0.0 -> (none)
- joint base_r_passive_wheel_x_frame_joint: origin xyz=0.1495                 -0.055                 0.03 rpy=0.0 0.0 0.0 -> (none)
- joint base_range_sensor_joint: origin xyz=0.1675 0.0 0.1844 rpy=0.0 0.0 0.0 -> (none)
- joint hand_camera_frame_joint: origin xyz=0.039 0.0 -0.0045 rpy=0.0 0.0 0.0 -> (none)
- joint hand_camera_gazebo_frame_joint: origin xyz=0 0 0 rpy=1.5707963268 -1.5707963268 0 -> xyz=0 0 0 rpy=1.570796326795 -1.570796326795 0
- joint hand_l_distal_joint: axis 1.0 0.0 0.0 -> (none)
- joint hand_l_finger_tip_frame_joint: origin xyz=0.01675 0.0193 0.0379 rpy=-1.5707963268 0.0 0.0 -> xyz=0.01675 0.0193 0.0379 rpy=-1.570796326795 0.0 0.0
- joint hand_l_finger_vacuum_frame_joint: origin xyz=0.00475 -0.011539 0.03322 rpy=0.785398163398 0.0 0.0 -> xyz=0.00475 -0.011539 0.03322 rpy=0.7853981633975 0.0 0.0
- joint hand_l_mimic_distal_joint: axis 1.0 0.0 0.0 -> (none); origin xyz=0.0 0.0 0.07 -> (none)
- joint hand_l_proximal_joint: axis 1.0 0.0 0.0 -> (none); origin xyz=-0.01675 -0.0245 -0.0175 rpy=0.0 0.0 0.0 -> (none)
- joint hand_l_spring_proximal_joint: axis 1.0 0.0 0.0 -> (none)
- joint hand_palm_joint: origin xyz=0.012 0.0 0.1405 rpy=0.0 0.0 3.14159265359 -> (none)
- joint hand_r_distal_joint: axis -1.0 0.0 0.0 -> (none)
- joint hand_r_finger_tip_frame_joint: origin xyz=0.01675 -0.0193 0.0379 rpy=1.5707963268 0.0 0.0 -> xyz=0.01675 -0.0193 0.0379 rpy=1.570796326795 0.0 0.0
- joint hand_r_mimic_distal_joint: axis -1.0 0.0 0.0 -> (none); origin xyz=0.0 0.0 0.07 -> (none)
- joint hand_r_proximal_joint: axis -1.0 0.0 0.0 -> (none); origin xyz=-0.01675 0.0245 -0.0175 rpy=0.0 0.0 0.0 -> (none)
- joint hand_r_spring_proximal_joint: axis -1.0 0.0 0.0 -> (none)
- joint head_center_camera_frame_joint: origin xyz=0.0195 0.0 0.061 rpy=-1.5707963268 0.0 -1.5707963268 -> (none)
- joint head_center_camera_gazebo_frame_joint: origin xyz=0 0 0 rpy=1.5707963268 -1.5707963268 0.0 -> xyz=0 0 0 rpy=1.570796326795 -1.570796326795 0.0
- joint head_l_stereo_camera_gazebo_frame_joint: origin xyz=0 0 0 rpy=1.5707963268 -1.5707963268 0.0 -> xyz=0 0 0 rpy=1.570796326795 -1.570796326795 0.0
- joint head_l_stereo_camera_joint: origin xyz=0.02 0.07 0.061 rpy=-1.5707963268 0.0 -1.5707963268 -> (none)
- joint head_pan_joint: origin xyz=0.0 0.0 0.0 rpy=0.0 0.0 0.0 -> (none)
- joint head_r_stereo_camera_gazebo_frame_joint: origin xyz=0 0 0 rpy=1.5707963268 -1.5707963268 0.0 -> xyz=0 0 0 rpy=1.570796326795 -1.570796326795 0.0
- joint head_r_stereo_camera_joint: origin xyz=0.02 -0.07 0.061 rpy=-1.5707963268 0.0 -1.5707963268 -> (none)
- joint head_rgbd_sensor_gazebo_frame_joint: origin xyz=0 0 0 rpy=1.5707963268 -1.5707963268 0.0 -> xyz=0 0 0 rpy=1.570796326795 -1.570796326795 0.0
- joint head_rgbd_sensor_joint: origin xyz=-0.079796 0.022 0.215172 rpy=-1.5707963268 0.0 -1.5707963268 -> (none)
- joint torso_lift_joint: origin xyz=0.0 0.0 0.752 rpy=0.0 0.0 0.0 -> (none)
- joint wrist_ft_sensor_frame_joint: origin xyz=0.0 0.0 0.0735 rpy=3.14159265359 0.0 0.0 -> (none)

File: robots/hsrb4s.urdf.xacro (robot description, xacro)
@@ -29,5 +29,5 @@
        xmlns:interface="http://playerstage.sourceforge.net/gazebo/xmlschema/#interface"
        xmlns:sensor="http://playerstage.sourceforge.net/gazebo/xmlschema/#sensor"
-       xmlns:xacro="http://ros.org/wiki/xacro">
+       xmlns:xacro="http://www.ros.org/wiki.xacro">
     <!-- common xacro -->
     <xacro:include filename="$(find hsr_description)/urdf/common.xacro" />
@@ -40,13 +40,8 @@
     <xacro:include filename="$(find hsr_description)/urdf/wrist_v0/wrist.urdf.xacro" />
     <xacro:include filename="$(find hsr_description)/urdf/hand_v0/hand.urdf.xacro" />
-    <!-- This switches a format of mesh files for visual property -->
-    <xacro:arg name="use_obj_for_visual" default="false" />
-    <xacro:arg name="use_obj_for_collision" default="false" />
-    <xacro:property name="g_use_obj_for_visual" value="$(arg use_obj_for_visual)"/>
-    <xacro:property name="g_use_obj_for_collision" value="$(arg use_obj_for_collision)"/>
     <!-- constant -->
-    <xacro:property name="g_robot_name" value="hsrb"/>
+    <xacro:property name="robot_name" value="hsrb"/>
     <!-- create robot -->
-    <xacro:hsrb_base prefix="base" robot_namespace="${g_robot_name}"/>
+    <xacro:hsrb_base prefix="base" robot_namespace="${robot_name}"/>
     <xacro:hsrb_torso prefix="torso" parent="base_link" mimic_joint="arm_lift_joint">
         <origin xyz="0.0 0.0 0.752" rpy="0.0 0.0 0.0"/>
@@ -58,5 +53,5 @@
         <origin xyz="0.0 0.0 0.340" rpy="0.0 0.0 0.0"/>
     </xacro:hsrb_arm>
-    <xacro:hsrb_wrist prefix="wrist" parent="arm_roll_link" robot_namespace="${g_robot_name}">
+    <xacro:hsrb_wrist prefix="wrist" parent="arm_roll_link" robot_namespace="${robot_name}">
         <origin xyz="0.0 0.0 0.0" rpy="0.0 0.0 0.0"/>
     </xacro:hsrb_wrist>
@@ -65,9 +60,9 @@
     </xacro:hsrb_hand>
     <gazebo>
-        <plugin name="${g_robot_name}_ros_control" filename="lib${g_robot_name}_gazebo_ros_control.so">
-            <robotNamespace>${g_robot_name}</robotNamespace>
+        <plugin name="${robot_name}_ros_control" filename="lib${robot_name}_gazebo_ros_control.so">
+            <robotNamespace>${robot_name}</robotNamespace>
         </plugin>
-        <plugin name="${g_robot_name}_p3d_ground_truth" filename="libgazebo_ros_p3d.so">
-            <robotNamespace>${g_robot_name}</robotNamespace>
+        <plugin name="${robot_name}_p3d_ground_truth" filename="libgazebo_ros_p3d.so">
+            <robotNamespace>${robot_name}</robotNamespace>
             <bodyName>base_footprint</bodyName>
             <topicName>odom_ground_truth</topicName>

File: urdf/arm_v0/arm.urdf.xacro (robot description, xacro)
@@ -47,20 +47,10 @@
             <visual>
                 <geometry>
-                    <xacro:unless value="${g_use_obj_for_visual}">
-                        <mesh filename="package://hsr_meshes/meshes/arm_v0/shoulder.dae" />
-                    </xacro:unless>
-                    <xacro:if value="${g_use_obj_for_visual}">
-                        <mesh filename="package://hsr_meshes/meshes/arm_v0/shoulder.obj" />
-                    </xacro:if>
+                    <mesh filename="package://hsr_meshes/meshes/arm_v0/shoulder.dae" />
                 </geometry>
             </visual>
             <collision>
                 <geometry>
-                    <xacro:unless value="${g_use_obj_for_collision}">
-                        <mesh filename="package://hsr_meshes/meshes/arm_v0/shoulder.stl" />
-                    </xacro:unless>
-                    <xacro:if value="${g_use_obj_for_collision}">
-                        <mesh filename="package://hsr_meshes/meshes/arm_v0/shoulder.collision.obj" />
-                    </xacro:if>
+                    <mesh filename="package://hsr_meshes/meshes/arm_v0/shoulder.stl" />
                 </geometry>
             </collision>
@@ -77,25 +67,16 @@
             <inertial>
                 <mass value="1.339295"/>
-                <origin xyz="-0.000459 0.006583 0.106069"/>
-                <inertia ixx="0.00889053" ixy="0.0" ixz="0.0" iyy="0.00825549" iyz="0.0" izz="0.00190511"/>
+                <origin xyz="0.000632 0.006404 0.118529"/>
+                <inertia ixx="7.528" ixy="-0.000020284207" ixz="-0.000022947194"
+                    iyy="0.007102" iyz="-0.000091796075" izz="0.001552"/>
             </inertial>
             <visual>
                 <geometry>
-                    <xacro:unless value="${g_use_obj_for_visual}">
-                        <mesh filename="package://hsr_meshes/meshes/arm_v0/arm_flex_light.dae" />
-                    </xacro:unless>
-                    <xacro:if value="${g_use_obj_for_visual}">
-                        <mesh filename="package://hsr_meshes/meshes/arm_v0/arm_flex_light.obj" />
-                    </xacro:if>
+                    <mesh filename="package://hsr_meshes/meshes/arm_v0/arm_flex_light.dae" />
                 </geometry>
             </visual>
             <collision>
                 <geometry>
-                    <xacro:unless value="${g_use_obj_for_collision}">
-                        <mesh filename="package://hsr_meshes/meshes/arm_v0/arm_flex.stl" />
-                    </xacro:unless>
-                    <xacro:if value="${g_use_obj_for_collision}">
-                        <mesh filename="package://hsr_meshes/meshes/arm_v0/arm_flex.collision.obj" />
-                    </xacro:if>
+                    <mesh filename="package://hsr_meshes/meshes/arm_v0/arm_flex.stl" />
                 </geometry>
             </collision>
@@ -118,20 +99,10 @@
             <visual>
                 <geometry>
-                    <xacro:unless value="${g_use_obj_for_visual}">
-                        <mesh filename="package://hsr_meshes/meshes/arm_v0/arm_roll_light.dae" />
-                    </xacro:unless>
-                    <xacro:if value="${g_use_obj_for_visual}">
-                        <mesh filename="package://hsr_meshes/meshes/arm_v0/arm_roll_light.obj" />
-                    </xacro:if>
+                    <mesh filename="package://hsr_meshes/meshes/arm_v0/arm_roll_light.dae" />
                 </geometry>
             </visual>
             <collision>
                 <geometry>
-                    <xacro:unless value="${g_use_obj_for_collision}">
-                        <mesh filename="package://hsr_meshes/meshes/arm_v0/arm_roll.stl" />
-                    </xacro:unless>
-                    <xacro:if value="${g_use_obj_for_collision}">
-                        <mesh filename="package://hsr_meshes/meshes/arm_v0/arm_roll.collision.obj" />
-                    </xacro:if>
+                    <mesh filename="package://hsr_meshes/meshes/arm_v0/arm_roll.stl" />
                 </geometry>
             </collision>

File: urdf/base_v2/base.urdf.xacro (robot description, xacro)
@@ -144,41 +144,21 @@
             <visual>
                 <geometry>
-                    <xacro:unless value="${g_use_obj_for_visual}">
-                        <mesh filename="package://hsr_meshes/meshes/base_v2/base_light.dae" />
-                    </xacro:unless>
-                    <xacro:if value="${g_use_obj_for_visual}">
-                        <mesh filename="package://hsr_meshes/meshes/base_v2/base_light.obj" />
-                    </xacro:if>
-                </geometry>
-            </visual>
-            <visual>
-                <geometry>
-                    <xacro:unless value="${g_use_obj_for_visual}">
-                        <mesh filename="package://hsr_meshes/meshes/base_v2/body_light.dae" />
-                    </xacro:unless>
-                    <xacro:if value="${g_use_obj_for_visual}">
-                        <mesh filename="package://hsr_meshes/meshes/base_v2/body_light.obj" />
-                    </xacro:if>
-                </geometry>
-            </visual>
-            <visual>
-                <geometry>
-                    <xacro:unless value="${g_use_obj_for_visual}">
-                        <mesh filename="package://hsr_meshes/meshes/base_v2/torso_base.dae" />
-                    </xacro:unless>
-                    <xacro:if value="${g_use_obj_for_visual}">
-                        <mesh filename="package://hsr_meshes/meshes/base_v2/torso_base.obj" />
-                    </xacro:if>
+                    <mesh filename="package://hsr_meshes/meshes/base_v2/base_light.dae" />
+                </geometry>
+            </visual>
+            <visual>
+                <geometry>
+                    <mesh filename="package://hsr_meshes/meshes/base_v2/body_light.dae" />
+                </geometry>
+            </visual>
+            <visual>
+                <geometry>
+                    <mesh filename="package://hsr_meshes/meshes/base_v2/torso_base.dae" />
                 </geometry>
             </visual>
             <collision>
                 <geometry>
-                    <xacro:unless value="${g_use_obj_for_collision}">
-                        <mesh filename="package://hsr_meshes/meshes/base_v2/base.stl" />
-	            </xacro:unless>
-		    <xacro:if value="${g_use_obj_for_collision}">
-			<mesh filename="package://hsr_meshes/meshes/base_v2/base.collision.obj" />
-                    </xacro:if>
-		</geometry>
+                    <mesh filename="package://hsr_meshes/meshes/base_v2/base.stl" />
+                </geometry>
             </collision>
         </link>

File: urdf/common.xacro (robot description, xacro)
@@ -28,5 +28,5 @@
   <xacro:arg name="implicit_damping" default="false" />
   <xacro:property name="pi" value="3.14159265359"/>
-  <macro name="hsrb_position_joint_transmission" params="joint reduction">
+  <xacro:macro name="hsrb_position_joint_transmission" params="joint reduction">
      <transmission name="${joint}_transmission">
        <type>transmission_interface/SimpleTransmission</type>
@@ -39,6 +39,6 @@
        </actuator>
      </transmission>
-  </macro>
-  <macro name="hsrb_effort_joint_transmission" params="joint reduction">
+  </xacro:macro>
+  <xacro:macro name="hsrb_effort_joint_transmission" params="joint reduction">
      <transmission name="${joint}_transmission">
        <type>transmission_interface/SimpleTransmission</type>
@@ -51,6 +51,6 @@
        </actuator>
      </transmission>
-  </macro>
-  <macro name="hsrb_velocity_joint_transmission" params="joint reduction">
+  </xacro:macro>
+  <xacro:macro name="hsrb_velocity_joint_transmission" params="joint reduction">
       <transmission name="${prefix}_transmission">
           <type>transmission_interface/SimpleTransmission</type>
@@ -63,6 +63,6 @@
           </actuator>
       </transmission>
-  </macro>
-  <macro name="gazebo_link" params="name gravity collide friction">
+  </xacro:macro>
+  <xacro:macro name="gazebo_link" params="name gravity collide friction">
     <gazebo reference="${name}">
       <selfCollide>${collide}</selfCollide>
@@ -71,6 +71,6 @@
       <mu2>${friction}</mu2>
     </gazebo>
-  </macro>
-  <macro name="gazebo_link_flat_black" params="name gravity collide friction">
+  </xacro:macro>
+  <xacro:macro name="gazebo_link_flat_black" params="name gravity collide friction">
     <gazebo reference="${name}">
       <selfCollide>${collide}</selfCollide>
@@ -80,6 +80,6 @@
       <material value="Gazebo/FlatBlack"/>
     </gazebo>
-  </macro>
-  <macro name="gazebo_link_caster" params="name">
+  </xacro:macro>
+  <xacro:macro name="gazebo_link_caster" params="name">
     <gazebo reference="${name}">
       <selfCollide>false</selfCollide>
@@ -90,6 +90,6 @@
       <material value="Gazebo/FlatBlack"/>
     </gazebo>
-  </macro>
-  <macro name="gazebo_link_rubber" params="name">
+  </xacro:macro>
+  <xacro:macro name="gazebo_link_rubber" params="name">
     <gazebo reference="${name}">
       <selfCollide>false</selfCollide>
@@ -105,6 +105,6 @@
       <material value="Gazebo/FlatBlack"/>
     </gazebo>
-  </macro>
-  <macro name="gazebo_joint" params="name">
+  </xacro:macro>
+  <xacro:macro name="gazebo_joint" params="name">
     <gazebo reference="${name}">
       <xacro:if value="$(arg implicit_damping)">
@@ -112,8 +112,8 @@
       </xacro:if>
     </gazebo>
-  </macro>
-  <macro name="gazebo_joint_mimic" params="name">
+  </xacro:macro>
+  <xacro:macro name="gazebo_joint_mimic" params="name">
     <gazebo reference="${name}">
     </gazebo>
-  </macro>
+  </xacro:macro>
 </robot>
