Commit message: [UPD] description

File: urdf/hand_v0/hand.urdf.xacro (robot description, xacro)
@@ -65,21 +65,11 @@
             <visual>
                 <geometry>
-                    <xacro:unless value="${g_use_obj_for_visual}">
-                        <mesh filename="package://hsr_meshes/meshes/hand_v0/palm.stl" />
-                    </xacro:unless>
-                    <xacro:if value="${g_use_obj_for_visual}">
-                        <mesh filename="package://hsr_meshes/meshes/hand_v0/palm.obj" />
-                    </xacro:if>
-                </geometry>
-                <material name="body_sub" />
-            </visual>
-            <collision>
-                <geometry>
-                    <xacro:unless value="${g_use_obj_for_collision}">
-                        <mesh filename="package://hsr_meshes/meshes/hand_v0/palm.stl" />
-                    </xacro:unless>
-                    <xacro:if value="${g_use_obj_for_collision}">
-                        <mesh filename="package://hsr_meshes/meshes/hand_v0/palm.obj" />
-                    </xacro:if>
+                    <mesh filename="package://hsr_meshes/meshes/hand_v0/palm.stl" />
+                </geometry>
+                <material name="body_sub" />
+            </visual>
+            <collision>
+                <geometry>
+                    <mesh filename="package://hsr_meshes/meshes/hand_v0/palm.stl" />
                 </geometry>
             </collision>
@@ -110,5 +100,5 @@
         </xacro:hsrb_finger_without_vacuum>
         <!-- camera -->
-        <xacro:wide_camera prefix="${prefix}" parent="${prefix}_palm_link" robot_namespace="${g_robot_name}" rpy="${pi/2.0} ${-pi/2.0} 0" >
+        <xacro:wide_camera prefix="${prefix}" parent="${prefix}_palm_link" robot_namespace="${robot_name}" rpy="${pi/2.0} ${-pi/2.0} 0" >
             <origin xyz="0.039 0.0 -0.0045" rpy="0.0 0.0 0.0"/>
         </xacro:wide_camera>
@@ -183,21 +173,11 @@
             <visual>
                 <geometry>
-                    <xacro:unless value="${g_use_obj_for_visual}">
-                        <mesh filename="package://hsr_meshes/meshes/hand_v0/l_proximal.stl" />
-                    </xacro:unless>
-                    <xacro:if value="${g_use_obj_for_visual}">
-                        <mesh filename="package://hsr_meshes/meshes/hand_v0/l_proximal.obj" />
-                    </xacro:if>
-                </geometry>
-                <material name="body_sub" />
-            </visual>
-            <collision>
-                <geometry>
-                    <xacro:unless value="${g_use_obj_for_collision}">
-                        <mesh filename="package://hsr_meshes/meshes/hand_v0/l_proximal.stl" />
-                    </xacro:unless>
-                    <xacro:if value="${g_use_obj_for_collision}">
-                        <mesh filename="package://hsr_meshes/meshes/hand_v0/l_proximal.obj" />
-                    </xacro:if>
+                    <mesh filename="package://hsr_meshes/meshes/hand_v0/l_proximal.stl" />
+                </geometry>
+                <material name="body_sub" />
+            </visual>
+            <collision>
+                <geometry>
+                    <mesh filename="package://hsr_meshes/meshes/hand_v0/l_proximal.stl" />
                 </geometry>
             </collision>
@@ -212,26 +192,16 @@
                 <origin xyz="0.011116 0.005679 0.017532"/>
                 <inertia
-                    ixx="0.000004451952" ixy="0.0" ixz="0.0"
-                    iyy="0.000000503765" iyz="0.0" izz="0.000004456764"/>
-            </inertial>
-            <visual>
-                <geometry>
-                    <xacro:unless value="${g_use_obj_for_visual}">
-                        <mesh filename="package://hsr_meshes/meshes/hand_v0/l_distal.stl" />
-                    </xacro:unless>
-                    <xacro:if value="${g_use_obj_for_visual}">
-                        <mesh filename="package://hsr_meshes/meshes/hand_v0/l_distal.obj" />
-                    </xacro:if>
-                </geometry>
-                <material name="body_sub" />
-            </visual>
-            <collision>
-                <geometry>
-                    <xacro:unless value="${g_use_obj_for_collision}">
-                        <mesh filename="package://hsr_meshes/meshes/hand_v0/l_distal.stl" />
-                    </xacro:unless>
-                    <xacro:if value="${g_use_obj_for_collision}">
-                        <mesh filename="package://hsr_meshes/meshes/hand_v0/l_distal.obj" />
-                    </xacro:if>
+                    ixx="0.000004451952" ixy="-0.000000617574" ixz="0.000000503765"
+                    iyy="0.000000503765" iyz="-0.000000435048" izz="0.000004456764"/>
+            </inertial>
+            <visual>
+                <geometry>
+                    <mesh filename="package://hsr_meshes/meshes/hand_v0/l_distal.stl" />
+                </geometry>
+                <material name="body_sub" />
+            </visual>
+            <collision>
+                <geometry>
+                    <mesh filename="package://hsr_meshes/meshes/hand_v0/l_distal.stl" />
                 </geometry>
             </collision>
@@ -281,21 +251,11 @@
             <visual>
                 <geometry>
-                    <xacro:unless value="${g_use_obj_for_visual}">
-                        <mesh filename="package://hsr_meshes/meshes/hand_v0/r_proximal.stl" />
-                    </xacro:unless>
-                    <xacro:if value="${g_use_obj_for_visual}">
-                        <mesh filename="package://hsr_meshes/meshes/hand_v0/r_proximal.obj" />
-                    </xacro:if>
-                </geometry>
-                <material name="body_sub" />
-            </visual>
-            <collision>
-                <geometry>
-                    <xacro:unless value="${g_use_obj_for_collision}">
-                        <mesh filename="package://hsr_meshes/meshes/hand_v0/r_proximal.stl" />
-                    </xacro:unless>
-                    <xacro:if value="${g_use_obj_for_collision}">
-                        <mesh filename="package://hsr_meshes/meshes/hand_v0/r_proximal.obj" />
-                    </xacro:if>
+                    <mesh filename="package://hsr_meshes/meshes/hand_v0/r_proximal.stl" />
+                </geometry>
+                <material name="body_sub" />
+            </visual>
+            <collision>
+                <geometry>
+                    <mesh filename="package://hsr_meshes/meshes/hand_v0/r_proximal.stl" />
                 </geometry>
             </collision>
@@ -315,21 +275,11 @@
             <visual>
                 <geometry>
-                    <xacro:unless value="${g_use_obj_for_visual}">
-                        <mesh filename="package://hsr_meshes/meshes/hand_v0/r_distal.stl" />
-                    </xacro:unless>
-                    <xacro:if value="${g_use_obj_for_visual}">
-                        <mesh filename="package://hsr_meshes/meshes/hand_v0/r_distal.obj" />
-                    </xacro:if>
-                </geometry>
-                <material name="body_sub" />
-            </visual>
-            <collision>
-                <geometry>
-                    <xacro:unless value="${g_use_obj_for_collision}">
-                        <mesh filename="package://hsr_meshes/meshes/hand_v0/r_distal.stl" />
-                    </xacro:unless>
-                    <xacro:if value="${g_use_obj_for_collision}">
-                        <mesh filename="package://hsr_meshes/meshes/hand_v0/r_distal.obj" />
-                    </xacro:if>
+                    <mesh filename="package://hsr_meshes/meshes/hand_v0/r_distal.stl" />
+                </geometry>
+                <material name="body_sub" />
+            </visual>
+            <collision>
+                <geometry>
+                    <mesh filename="package://hsr_meshes/meshes/hand_v0/r_distal.stl" />
                 </geometry>
             </collision>

File: urdf/head_v2/head.urdf.xacro (robot description, xacro)
@@ -50,20 +50,10 @@
             <visual>
                 <geometry>
-                    <xacro:unless value="${g_use_obj_for_visual}">
-                        <mesh filename="package://hsr_meshes/meshes/head_v1/head_pan.dae" />
-                    </xacro:unless>
-                    <xacro:if value="${g_use_obj_for_visual}">
-                        <mesh filename="package://hsr_meshes/meshes/head_v1/head_pan.obj" />
-                    </xacro:if>
+                    <mesh filename="package://hsr_meshes/meshes/head_v1/head_pan.dae" />
                 </geometry>
             </visual>
             <collision>
                 <geometry>
-                    <xacro:unless value="${g_use_obj_for_collision}">
-                        <mesh filename="package://hsr_meshes/meshes/head_v1/head_pan.stl" />
-                    </xacro:unless>
-                    <xacro:if value="${g_use_obj_for_collision}">
-                        <mesh filename="package://hsr_meshes/meshes/head_v1/head_pan.obj" />
-                    </xacro:if>
+                    <mesh filename="package://hsr_meshes/meshes/head_v1/head_pan.stl" />
                 </geometry>
             </collision>
@@ -86,64 +76,39 @@
             <visual>
                 <geometry>
-                    <xacro:unless value="${g_use_obj_for_visual}">
-                        <mesh filename="package://hsr_meshes/meshes/head_v1/head_upper.dae" />
-                    </xacro:unless>
-                    <xacro:if value="${g_use_obj_for_visual}">
-                        <mesh filename="package://hsr_meshes/meshes/head_v1/head_upper.obj" />
-                    </xacro:if>
+                    <mesh filename="package://hsr_meshes/meshes/head_v1/head_upper.dae" />
                 </geometry>
             </visual>
             <visual>
                 <geometry>
-                    <xacro:unless value="${g_use_obj_for_visual}">
-                        <mesh filename="package://hsr_meshes/meshes/head_v1/head_tilt.dae" />
-                    </xacro:unless>
-                    <xacro:if value="${g_use_obj_for_visual}">
-                        <mesh filename="package://hsr_meshes/meshes/head_v1/head_tilt.obj" />
-                    </xacro:if>
+                    <mesh filename="package://hsr_meshes/meshes/head_v1/head_tilt.dae" />
                 </geometry>
             </visual>
             <visual>
                 <geometry>
-                    <xacro:unless value="${g_use_obj_for_visual}">
-                        <mesh filename="package://hsr_meshes/meshes/head_v1/tablet_base.dae" />
-                    </xacro:unless>
-                    <xacro:if value="${g_use_obj_for_visual}">
-                        <mesh filename="package://hsr_meshes/meshes/head_v1/tablet_base.obj" />
-                    </xacro:if>
+                    <mesh filename="package://hsr_meshes/meshes/head_v1/tablet_base.dae" />
                 </geometry>
             </visual>
             <collision>
                 <geometry>
-                    <xacro:unless value="${g_use_obj_for_collision}">
-                        <mesh filename="package://hsr_meshes/meshes/head_v1/head.stl" />
-                    </xacro:unless>
-                    <xacro:if value="${g_use_obj_for_collision}">
-                        <mesh filename="package://hsr_meshes/meshes/head_v1/head.obj" />
-                    </xacro:if>
+                    <mesh filename="package://hsr_meshes/meshes/head_v1/head.stl" />
                 </geometry>
             </collision>
             <collision>
                 <geometry>
-                    <xacro:unless value="${g_use_obj_for_collision}">
-                        <mesh filename="package://hsr_meshes/meshes/head_v1/tablet.stl" />
-                    </xacro:unless>
-                    <xacro:if value="${g_use_obj_for_collision}">
-                        <mesh filename="package://hsr_meshes/meshes/head_v1/tablet.obj" />
-                    </xacro:if>
+                    <mesh filename="package://hsr_meshes/meshes/head_v1/tablet.stl" />
                 </geometry>
             </collision>
         </link>
         <!-- cameras -->
-        <xacro:rgb_sensor prefix="${prefix}_l_stereo" parent="${prefix}_tilt_link" robot_namespace="${g_robot_name}" baseline="0.00">
+        <xacro:rgb_sensor prefix="${prefix}_l_stereo" parent="${prefix}_tilt_link" robot_namespace="${robot_name}" baseline="0.00">
             <origin xyz="0.02 0.07 0.061" rpy="${-pi/2.0} 0.0 ${-pi/2.0}"/>
         </xacro:rgb_sensor>
-        <xacro:rgb_sensor prefix="${prefix}_r_stereo" parent="${prefix}_tilt_link" robot_namespace="${g_robot_name}" baseline="0.14">
+        <xacro:rgb_sensor prefix="${prefix}_r_stereo" parent="${prefix}_tilt_link" robot_namespace="${robot_name}" baseline="0.14">
             <origin xyz="0.02 -0.07 0.061" rpy="${-pi/2.0} 0.0 ${-pi/2.0}"/>
         </xacro:rgb_sensor>
-        <xacro:wide_camera prefix="${prefix}_center" parent="${prefix}_tilt_link" robot_namespace="${g_robot_name}" rpy="${pi/2.0} ${-pi/2.0} 0.0" >
+        <xacro:wide_camera prefix="${prefix}_center" parent="${prefix}_tilt_link" robot_namespace="${robot_name}" rpy="${pi/2.0} ${-pi/2.0} 0.0" >
             <origin xyz="0.0195 0.0 0.061" rpy="${-pi/2.0} 0.0 ${-pi/2.0}"/>
         </xacro:wide_camera>
-        <xacro:rgbd_sensor prefix="${prefix}" parent="${prefix}_tilt_link" robot_namespace="${g_robot_name}" sensor_name="rgbd_sensor">
+        <xacro:rgbd_sensor prefix="${prefix}" parent="${prefix}_tilt_link" robot_namespace="${robot_name}" sensor_name="rgbd_sensor">
             <origin xyz="-0.079796 0.022 0.215172" rpy="${-pi/2.0} 0.0 ${-pi/2.0}"/>
         </xacro:rgbd_sensor>

File: urdf/materials.urdf.xacro (robot description, xacro)
@@ -30,5 +30,5 @@
   </material>
   <material name="body_sub">
-    <color rgba="0.3333 0.3333 0.3333 1.0"/>
+    <color rgba="0.33 0.33 0.33 1.0"/>
   </material>
   <material name="wheel">

File: urdf/sensors/laser.urdf.xacro (robot description, xacro)
@@ -37,20 +37,10 @@
             <visual>
                 <geometry>
-                    <xacro:unless value="${g_use_obj_for_visual}">
-                        <mesh filename="package://hsr_meshes/meshes/sensors/laser.dae" />
-                    </xacro:unless>
-                    <xacro:if value="${g_use_obj_for_visual}">
-                        <mesh filename="package://hsr_meshes/meshes/sensors/laser.obj" />
-                    </xacro:if>
+                    <mesh filename="package://hsr_meshes/meshes/sensors/laser.dae" />
                 </geometry>
             </visual>
             <collision>
                 <geometry>
-                    <xacro:unless value="${g_use_obj_for_collision}">
-                        <mesh filename="package://hsr_meshes/meshes/sensors/laser.stl" />
-                    </xacro:unless>
-                    <xacro:if value="${g_use_obj_for_collision}">
-                        <mesh filename="package://hsr_meshes/meshes/sensors/laser.obj" />
-                    </xacro:if>
+                    <mesh filename="package://hsr_meshes/meshes/sensors/laser.stl" />
                 </geometry>
             </collision>

File: urdf/sensors/rgb_sensor.urdf.xacro (robot description, xacro)
@@ -37,10 +37,5 @@
                 <origin xyz="0 0 0" rpy="0.0 0.0 0.0"/>
                 <geometry>
-                    <xacro:if value="${g_use_obj_for_visual}">
-                        <mesh filename="package://hsr_meshes/meshes/sensors/head_camera.obj" />
-                    </xacro:if>
-                    <xacro:unless value="${g_use_obj_for_visual}">
-                        <mesh filename="package://hsr_meshes/meshes/sensors/head_camera.dae" />
-                    </xacro:unless>
+                    <mesh filename="package://hsr_meshes/meshes/sensors/head_camera.dae" />
                 </geometry>
             </visual>

File: urdf/sensors/rgbd_sensor.urdf.xacro (robot description, xacro)
@@ -37,21 +37,11 @@
                 <origin xyz="0 0 0" rpy="0.0 0.0 0.0"/>
                 <geometry>
-                    <xacro:unless value="${g_use_obj_for_visual}">
-                        <mesh filename="package://hsr_meshes/meshes/sensors/rgbd_light.dae" />
-                    </xacro:unless>
-                    <xacro:if value="${g_use_obj_for_visual}">
-                        <mesh filename="package://hsr_meshes/meshes/sensors/rgbd_light.obj" />
-                    </xacro:if>
+                    <mesh filename="package://hsr_meshes/meshes/sensors/rgbd_light.dae" />
                 </geometry>
             </visual>
             <collision>
-               <origin xyz="0 0 0" rpy="0.0 0.0 0.0"/>
-               <geometry>
-                  <xacro:unless value="${g_use_obj_for_collision}">
-                     <mesh filename="package://hsr_meshes/meshes/sensors/rgbd.stl" />
-                  </xacro:unless>
-                  <xacro:if value="${g_use_obj_for_collision}">
-                     <mesh filename="package://hsr_meshes/meshes/sensors/rgbd.obj" />
-                  </xacro:if>
+                <origin xyz="0 0 0" rpy="0.0 0.0 0.0"/>
+                <geometry>
+                    <mesh filename="package://hsr_meshes/meshes/sensors/rgbd.stl" />
                 </geometry>
             </collision>

File: urdf/torso_v0/torso.urdf.xacro (robot description, xacro)
@@ -48,20 +48,10 @@
             <visual>
                 <geometry>
-                    <xacro:unless value="${g_use_obj_for_visual}">
-                        <mesh filename="package://hsr_meshes/meshes/torso_v0/torso_light.dae" />
-                    </xacro:unless>
-                    <xacro:if value="${g_use_obj_for_visual}">
-                        <mesh filename="package://hsr_meshes/meshes/torso_v0/torso_light.obj" />
-                    </xacro:if>
+                    <mesh filename="package://hsr_meshes/meshes/torso_v0/torso_light.dae" />
                 </geometry>
             </visual>
             <collision>
                 <geometry>
-                    <xacro:unless value="${g_use_obj_for_collision}">
-                        <mesh filename="package://hsr_meshes/meshes/torso_v0/torso.std" />
-                    </xacro:unless>
-                    <xacro:if value="${g_use_obj_for_collision}">
-                        <mesh filename="package://hsr_meshes/meshes/torso_v0/torso.collision.obj" />
-                    </xacro:if>
+                    <mesh filename="package://hsr_meshes/meshes/torso_v0/torso.stl" />
                 </geometry>
             </collision>

File: urdf/wrist_v0/wrist.urdf.xacro (robot description, xacro)
@@ -48,10 +48,5 @@
             <visual>
                 <geometry>
-                    <xacro:unless value="${g_use_obj_for_visual}">
-                        <mesh filename="package://hsr_meshes/meshes/wrist_v0/wrist_flex.dae" />
-                    </xacro:unless>
-                    <xacro:if value="${g_use_obj_for_visual}">
-                        <mesh filename="package://hsr_meshes/meshes/wrist_v0/wrist_flex.obj" />
-                    </xacro:if>
+                    <mesh filename="package://hsr_meshes/meshes/wrist_v0/wrist_flex.dae" />
                 </geometry>
                 <material name="body_sub" />
@@ -84,24 +79,14 @@
                 <origin xyz="-0.001416 -0.001547 0.081689"/>
                 <inertia ixx="0.000805633819" ixy="-0.000014431758" ixz="0.000028204659"
-                         iyy="0.000768077165" iyz="0.000022460226" izz="0.000453406611"/>
+                    iyy="0.000768077165" iyz="0.000022460226" izz="0.000453406611"/>
             </inertial>
             <visual>
                 <geometry>
-                    <xacro:unless value="${g_use_obj_for_visual}">
-                       <mesh filename="package://hsr_meshes/meshes/wrist_v0/wrist_roll.dae" />
-                    </xacro:unless>
-                    <xacro:if value="${g_use_obj_for_visual}">
-                       <mesh filename="package://hsr_meshes/meshes/wrist_v0/wrist_roll.obj" />
-                    </xacro:if>
+                    <mesh filename="package://hsr_meshes/meshes/wrist_v0/wrist_roll.dae" />
                 </geometry>
             </visual>
             <collision>
                 <geometry>
-                    <xacro:unless value="${g_use_obj_for_collision}">
-                      <mesh filename="package://hsr_meshes/meshes/wrist_v0/wrist_roll.stl" />
-                    </xacro:unless>
-                    <xacro:if value="${g_use_obj_for_collision}">
-                      <mesh filename="package://hsr_meshes/meshes/wrist_v0/wrist_roll.collision.obj" />
-                    </xacro:if>
+                    <mesh filename="package://hsr_meshes/meshes/wrist_v0/wrist_roll.stl" />
                 </geometry>
             </collision>
